File: MGBC PCB/MGBC-MBL-01_1-5_2.brd (EAGLE design)
At the start: 69.7 x 114.8 mm, 114 parts, among them P1 MGB-CART, P2 GBC_LCDH, P3 LINKPORTDMG-LINK-SHORT, P4 MGB-PWRJACK, P5 MGBHPMGB, Q2 3904, SW1 MGB-SW1, SW2 NAV_SWITCH, U1 GBC_CPU, U2 LH52256CVTXIZ, U3 LM4853, U4 TLV70233QDBVRQ1, U5 MGB-PWR_BD, U6 TPS3840, U7 TL331, X1 8.388608MHZ12SMX-B-4-PAD

Commit message: Add files via upload
Parts:
- C3: value 1u -> 100n
Changed lines of the file:
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@@
 <attribute name="VALUE" x="55.034" y="107.061" size="1.27" layer="27" rot="R180"/>
 </element>
-<element name="C3" library="rcl" package="C0603" package3d_urn="urn:adsk.eagle:package:23616/2" value="1u" x="58.101" y="105.156" smashed="yes">
+<element name="C3" library="rcl" package="C0603" package3d_urn="urn:adsk.eagle:package:23616/2" value="100n" x="58.101" y="105.156" smashed="yes">
 <attribute name="NAME" x="57.45975" y="105.9435" size="1" layer="25" font="vector" ratio="15"/>
 <attribute name="POPULARITY" value="37" x="58.101" y="105.156" size="1.778" layer="27" display="off"/>
